File: minimal_ltc3350/minimal_ltc3350.kicad_pcb (KiCad board)
At the start: 4 copper layers, 34.3 x 38.1 mm, 69 parts, among them Q1 20.0 V, Q2 20.0 V, Q3 20 V, Q4 20 V, Q5 20.0 V, U1 LTC3350EUHF-PBF

Commit message: Update KiCad project files: add new transistor components and connect nets
Parts:
- added Q6: 8 V, transistor_footprints:PowerPAK SC-70, F.Cu at (135.1, 100.3)
- added Q7: 8 V, transistor_footprints:PowerPAK SC-70, F.Cu at (127.3, 100.3)
- added Q8: 8 V, transistor_footprints:PowerPAK SC-70, F.Cu at (119.4, 100.3)
- added Q9: 8 V, transistor_footprints:PowerPAK SC-70, F.Cu at (111.5, 100.3)
- added R14: 2.7 Ω, resistor_footprints:R_2512_6332Metric, F.Cu at (137.7, 107.7)
- added R30: 2.7 Ω, resistor_footprints:R_2512_6332Metric, F.Cu at (137.7, 103.6)
- added R31: 2.7 Ω, resistor_footprints:R_2512_6332Metric, F.Cu at (129.8, 107.7)
- added R32: 2.7 Ω, resistor_footprints:R_2512_6332Metric, F.Cu at (129.8, 103.6)
- added R33: 2.7 Ω, resistor_footprints:R_2512_6332Metric, F.Cu at (121.9, 107.7)
- added R34: 2.7 Ω, resistor_footprints:R_2512_6332Metric, F.Cu at (121.9, 103.6)
- added R35: 2.7 Ω, resistor_footprints:R_2512_6332Metric, F.Cu at (114.0, 107.7)
- added R36: 2.7 Ω, resistor_footprints:R_2512_6332Metric, F.Cu at (114.0, 103.6)
- moved R23 21.3 mm to (111.5, 97.9), turned to 180 degrees
- moved R29 20.1 mm to (120.8, 87.5), turned to -90 degrees
- moved R28 17.0 mm to (124.9, 87.5), turned to -90 degrees
- moved R22 15.5 mm to (119.4, 97.9), turned to 180 degrees
- moved TP1 15.2 mm to (109.2, 77.5)
- moved TP2 15.2 mm to (109.2, 78.7)
- moved TP3 15.2 mm to (109.2, 80.0)
- moved TP4 15.2 mm to (109.2, 81.3)
- moved FID1 15.2 mm to (110.4, 110.6)
- moved FID2 15.2 mm to (110.4, 74.9)
- moved R21 9.82 mm to (127.3, 97.9), turned to 180 degrees
- moved Q5 7.74 mm to (121.7, 93.3), turned to 180 degrees
- moved R20 4.11 mm to (135.1, 97.9), turned to 180 degrees
Connections:
- R20 pad 2: unconnected-(R20-Pad2) -> Net-(Q6-S-Pad4)
- R21 pad 2: unconnected-(R21-Pad2) -> Net-(Q7-S-Pad4)
- R22 pad 2: unconnected-(R22-Pad2) -> Net-(Q8-S-Pad4)
Routing:
- net /CAPRTN: track 8.01 -> 30.2 mm
- net /CAP1: track 6.66 -> 22.4 mm
- net Net-(Q6-S-Pad4): track 0.00 -> 11.5 mm
- net Net-(Q8-S-Pad4): track 0.00 -> 11.5 mm
- net Net-(Q7-S-Pad4): track 0.00 -> 11.5 mm
- net /CAP2: track 5.97 -> 15.3 mm
- net Net-(Q9-D-Pad1): track 0.00 -> 7.26 mm
- net Net-(Q6-D-Pad1): track 0.00 -> 7.26 mm
- net Net-(Q8-D-Pad1): track 0.00 -> 7.26 mm
- net Net-(Q7-D-Pad1): track 0.00 -> 7.26 mm
- net Net-(Q5-S): track 0.00 -> 5.93 mm
- net /CAP3: track 6.32 -> 8.56 mm
- net /ITST: track 16.9 -> 18.1 mm
Other:
- board size 34.3 x 38.1 mm -> 49.5 x 38.1 mm
